Commit message: 代价地图无法显示，覆盖率差点意思

File: indoor_cartographer_demo/urdf/indoor_mapper_bot.urdf.xacro (robot description, xacro)
@@ -1,10 +1,10 @@
 <?xml version="1.0"?>
 <robot name="indoor_mapper_bot" xmlns:xacro="http://ros.org/wiki/xacro">
-  <xacro:property name="base_length" value="0.44" />
-  <xacro:property name="base_width" value="0.34" />
-  <xacro:property name="base_height" value="0.16" />
-  <xacro:property name="wheel_radius" value="0.08" />
-  <xacro:property name="wheel_width" value="0.045" />
-  <xacro:property name="wheel_y" value="0.215" />
+  <xacro:property name="base_length" value="0.34" />
+  <xacro:property name="base_width" value="0.25" />
+  <xacro:property name="base_height" value="0.13" />
+  <xacro:property name="wheel_radius" value="0.065" />
+  <xacro:property name="wheel_width" value="0.035" />
+  <xacro:property name="wheel_y" value="0.15" />
   <link name="base_footprint" />
   <joint name="base_footprint_joint" type="fixed">
@@ -15,7 +15,7 @@
   <link name="base_link">
     <inertial>
-      <origin xyz="0 0 0.08" />
-      <mass value="4.5" />
-      <inertia ixx="0.036" ixy="0" ixz="0" iyy="0.048" iyz="0" izz="0.064" />
+      <origin xyz="0 0 0.065" />
+      <mass value="3.2" />
+      <inertia ixx="0.020" ixy="0" ixz="0" iyy="0.028" iyz="0" izz="0.038" />
     </inertial>
     <visual>
@@ -29,5 +29,5 @@
     </visual>
     <collision name="base_collision">
-      <origin xyz="0 0 ${base_height / 2.0 + 0.015}" />
+      <origin xyz="0 0 ${base_height / 2.0 + 0.012}" />
       <geometry>
         <box size="${base_length} ${base_width} ${base_height}" />
@@ -37,6 +37,6 @@
   <link name="left_wheel_link">
     <inertial>
-      <mass value="0.45" />
-      <inertia ixx="0.0012" ixy="0" ixz="0" iyy="0.0012" iyz="0" izz="0.0012" />
+      <mass value="0.30" />
+      <inertia ixx="0.0007" ixy="0" ixz="0" iyy="0.0007" iyz="0" izz="0.0007" />
     </inertial>
     <visual>
@@ -58,6 +58,6 @@
   <link name="right_wheel_link">
     <inertial>
-      <mass value="0.45" />
-      <inertia ixx="0.0012" ixy="0" ixz="0" iyy="0.0012" iyz="0" izz="0.0012" />
+      <mass value="0.30" />
+      <inertia ixx="0.0007" ixy="0" ixz="0" iyy="0.0007" iyz="0" izz="0.0007" />
     </inertial>
     <visual>
@@ -82,5 +82,5 @@
     <visual>
       <geometry>
-        <sphere radius="0.035" />
+        <sphere radius="0.028" />
       </geometry>
       <material name="wheel_black" />
@@ -88,5 +88,5 @@
     <collision>
       <geometry>
-        <sphere radius="0.035" />
+        <sphere radius="0.028" />
       </geometry>
     </collision>
@@ -99,5 +99,5 @@
     <visual>
       <geometry>
-        <cylinder radius="0.058" length="0.05" />
+        <cylinder radius="0.045" length="0.04" />
       </geometry>
       <material name="laser_copper">
@@ -107,5 +107,5 @@
     <collision>
       <geometry>
-        <cylinder radius="0.058" length="0.05" />
+        <cylinder radius="0.045" length="0.04" />
       </geometry>
     </collision>
@@ -118,5 +118,5 @@
     <visual>
       <geometry>
-        <box size="0.04 0.07 0.045" />
+        <box size="0.035 0.055 0.035" />
       </geometry>
       <material name="camera_black">
@@ -126,5 +126,5 @@
     <collision>
       <geometry>
-        <box size="0.04 0.07 0.045" />
+        <box size="0.035 0.055 0.035" />
       </geometry>
     </collision>
@@ -145,15 +145,15 @@
     <parent link="base_link" />
     <child link="caster_link" />
-    <origin xyz="-0.17 0 0.035" />
+    <origin xyz="-0.13 0 0.028" />
   </joint>
   <joint name="laser_joint" type="fixed">
     <parent link="base_link" />
     <child link="laser_link" />
-    <origin xyz="0.11 0 0.235" />
+    <origin xyz="0.08 0 0.19" />
   </joint>
   <joint name="camera_joint" type="fixed">
     <parent link="base_link" />
     <child link="camera_link" />
-    <origin xyz="0.235 0 0.34" />
+    <origin xyz="0.185 0 0.27" />
   </joint>
   <gazebo reference="base_footprint">
@@ -254,6 +254,6 @@
       <wheelSeparation>${2.0 * wheel_y}</wheelSeparation>
       <wheelDiameter>${2.0 * wheel_radius}</wheelDiameter>
-      <wheelAcceleration>4.5</wheelAcceleration>
-      <wheelTorque>8</wheelTorque>
+      <wheelAcceleration>5.0</wheelAcceleration>
+      <wheelTorque>5</wheelTorque>
       <commandTopic>cmd_vel</commandTopic>
       <odometryTopic>odom</odometryTopic>

Commit message: 效果几乎完美的一版

File: indoor_cartographer_demo/urdf/indoor_mapper_bot.urdf.xacro (robot description, xacro)
@@ -1,10 +1,10 @@
 <?xml version="1.0"?>
 <robot name="indoor_mapper_bot" xmlns:xacro="http://ros.org/wiki/xacro">
-  <xacro:property name="base_length" value="0.34" />
-  <xacro:property name="base_width" value="0.25" />
-  <xacro:property name="base_height" value="0.13" />
-  <xacro:property name="wheel_radius" value="0.065" />
-  <xacro:property name="wheel_width" value="0.035" />
-  <xacro:property name="wheel_y" value="0.15" />
+  <xacro:property name="base_length" value="0.28" />
+  <xacro:property name="base_width" value="0.19" />
+  <xacro:property name="base_height" value="0.11" />
+  <xacro:property name="wheel_radius" value="0.055" />
+  <xacro:property name="wheel_width" value="0.03" />
+  <xacro:property name="wheel_y" value="0.125" />
   <link name="base_footprint" />
   <joint name="base_footprint_joint" type="fixed">
@@ -15,7 +15,7 @@
   <link name="base_link">
     <inertial>
-      <origin xyz="0 0 0.065" />
-      <mass value="3.2" />
-      <inertia ixx="0.020" ixy="0" ixz="0" iyy="0.028" iyz="0" izz="0.038" />
+      <origin xyz="0 0 0.055" />
+      <mass value="2.4" />
+      <inertia ixx="0.012" ixy="0" ixz="0" iyy="0.016" iyz="0" izz="0.022" />
     </inertial>
     <visual>
@@ -37,6 +37,6 @@
   <link name="left_wheel_link">
     <inertial>
-      <mass value="0.30" />
-      <inertia ixx="0.0007" ixy="0" ixz="0" iyy="0.0007" iyz="0" izz="0.0007" />
+      <mass value="0.22" />
+      <inertia ixx="0.00045" ixy="0" ixz="0" iyy="0.00045" iyz="0" izz="0.00045" />
     </inertial>
     <visual>
@@ -58,6 +58,6 @@
   <link name="right_wheel_link">
     <inertial>
-      <mass value="0.30" />
-      <inertia ixx="0.0007" ixy="0" ixz="0" iyy="0.0007" iyz="0" izz="0.0007" />
+      <mass value="0.22" />
+      <inertia ixx="0.00045" ixy="0" ixz="0" iyy="0.00045" iyz="0" izz="0.00045" />
     </inertial>
     <visual>
@@ -82,5 +82,5 @@
     <visual>
       <geometry>
-        <sphere radius="0.028" />
+        <sphere radius="0.024" />
       </geometry>
       <material name="wheel_black" />
@@ -88,5 +88,5 @@
     <collision>
       <geometry>
-        <sphere radius="0.028" />
+        <sphere radius="0.024" />
       </geometry>
     </collision>
@@ -99,5 +99,5 @@
     <visual>
       <geometry>
-        <cylinder radius="0.045" length="0.04" />
+        <cylinder radius="0.038" length="0.035" />
       </geometry>
       <material name="laser_copper">
@@ -107,5 +107,5 @@
     <collision>
       <geometry>
-        <cylinder radius="0.045" length="0.04" />
+        <cylinder radius="0.038" length="0.035" />
       </geometry>
     </collision>
@@ -129,4 +129,12 @@
       </geometry>
     </collision>
+  </link>
+  <link name="left_wing_link">
+    <inertial><mass value="0.015" /><inertia ixx="0.00002" ixy="0" ixz="0" iyy="0.00002" iyz="0" izz="0.00003" /></inertial>
+    <visual><geometry><box size="0.14 0.055 0.012" /></geometry><material name="wing_sky"><color rgba="0.20 0.72 0.95 1" /></material></visual>
+  </link>
+  <link name="right_wing_link">
+    <inertial><mass value="0.015" /><inertia ixx="0.00002" ixy="0" ixz="0" iyy="0.00002" iyz="0" izz="0.00003" /></inertial>
+    <visual><geometry><box size="0.14 0.055 0.012" /></geometry><material name="wing_sky" /></visual>
   </link>
   <joint name="left_wheel_joint" type="continuous">
@@ -145,15 +153,23 @@
     <parent link="base_link" />
     <child link="caster_link" />
-    <origin xyz="-0.13 0 0.028" />
+    <origin xyz="-0.105 0 0.024" />
   </joint>
   <joint name="laser_joint" type="fixed">
     <parent link="base_link" />
     <child link="laser_link" />
-    <origin xyz="0.08 0 0.19" />
+    <origin xyz="0.065 0 0.16" />
   </joint>
   <joint name="camera_joint" type="fixed">
     <parent link="base_link" />
     <child link="camera_link" />
-    <origin xyz="0.185 0 0.27" />
+    <origin xyz="0.15 0 0.23" />
+  </joint>
+  <joint name="left_wing_joint" type="fixed">
+    <parent link="base_link" /><child link="left_wing_link" />
+    <origin xyz="-0.015 0.105 0.145" rpy="0 0 0.45" />
+  </joint>
+  <joint name="right_wing_joint" type="fixed">
+    <parent link="base_link" /><child link="right_wing_link" />
+    <origin xyz="-0.015 -0.105 0.145" rpy="0 0 -0.45" />
   </joint>
   <gazebo reference="base_footprint">
@@ -184,4 +200,6 @@
     <mu2>1.0</mu2>
   </gazebo>
+  <gazebo reference="left_wing_link"><material>Gazebo/SkyBlue</material></gazebo>
+  <gazebo reference="right_wing_link"><material>Gazebo/SkyBlue</material></gazebo>
   <gazebo reference="laser_link">
     <material>Gazebo/Orange</material>
@@ -255,5 +273,5 @@
       <wheelDiameter>${2.0 * wheel_radius}</wheelDiameter>
       <wheelAcceleration>5.0</wheelAcceleration>
-      <wheelTorque>5</wheelTorque>
+      <wheelTorque>4</wheelTorque>
       <commandTopic>cmd_vel</commandTopic>
       <odometryTopic>odom</odometryTopic>
